File: cao_00/ex02/cao/cao.kicad_sch (KiCad schematic)
At the start: 8 parts, among them J2 AVR-ISP, U1 ATmega328P-AU, Y1 16MHz

Commit message: :arrow_up: feat: Update ex02
Parts:
- removed C1, C2: 22pF, symbol MyLibrary:Capacitors
- removed C4: 100nF, symbol MyLibrary:Capacitors
- removed C5: 10uF, symbol MyLibrary:Capacitors
- removed Y1: 16MHz, symbol MyLibrary:Crystal_Resonators
- added C1, C2: 22pF, symbol Device:C_Small
- added C4: 100nF, symbol Device:C_Small
- added C5: 10uF, symbol Device:C_Small
- added Y1: 16MHz, symbol Device:Crystal_GND2_Small
Connections:
- net +5V: now also C4.1, C5.1
- net GND: now also C1.1, C2.2, C4.2, C5.2, Y1.2
- net LED_0: now also U1.12 (PB0)
- net LED_1: now also U1.13 (PB1)
- net LED_2: now also U1.14 (PB2)
- net LED_3: now also U1.15 (PB3)
- net MISO: now also J2.1 (MISO)
- net MOSI: now also J2.4 (MOSI); no longer U1.15 (PB3)
- net SCK: now also J2.3 (SCK)
- net out: now also J2.5 (~{RST}), U1.1 (PD3), U1.29 (~{RESET}/PC6)
- net rx: now also U1.31 (PD1)
- net tx: now also U1.30 (PD0)
- net XTAL1: now reaches U1.7 (XTAL1/PB6)
- net XTAL1: now also C2.1, Y1.3
- net XTAL2: now reaches U1.8 (XTAL2/PB7)
- net XTAL2: now also C1.2, Y1.1
Other:
- removed sheet Sheet: led 0
- removed sheet Sheet: led 1
- removed sheet Sheet: led 2
- removed sheet Sheet: led 3
- added sheet Sheet: led_0 (led.kicad_sch)
- added sheet Sheet: led_1 (led.kicad_sch)
- added sheet Sheet: led_2 (led.kicad_sch)
- added sheet Sheet: led_3 (led.kicad_sch)
- sheet Sheet: button_but0: file untitled.kicad_sch -> button.kicad_sch
- sheet Sheet: button_reset: file untitled.kicad_sch -> button.kicad_sch
- sheet Sheet: usb_flasher: file untitled.kicad_sch -> usb_flasher.kicad_sch
- note removed: "LED_0"
- note removed: "LED_1"
- note removed: "LED_2"
- note removed: "LED_3"
